Commit message: set offsets for arm

File: urdf/ARMDIFF1.urdf (robot description, URDF)
Before this commit: robot ARMDIFF1, 6 links, 5 joints
Joints:
- joint linkOneJoint: origin xyz=0.08505 0 0.13572 rpy=0 0 0 -> xyz=0.08505 0 0.13572 rpy=0 2.17 0
- joint linkTwoJoint: origin xyz=-0.25101 0.0036996 0.34296 rpy=0 0 0 -> xyz=-0.25101 0.0036996 0.34296 rpy=0 -1.84 0
- joint rollJoint: origin xyz=0.017053 0 0.0065172 rpy=0 0 0 -> xyz=0.017053 0 0.0065172 rpy=0.4 0 0
