Commit message: urdf meshes update for rerun

File: urdf/rerun_ARMDIFF.urdf (robot description, URDF)
Before this commit: robot ARMDIFF1, 6 links, 5 joints
Links:
- link base_link: geometry collision mesh filename=~/Vibranium/baahubali/urdf/meshes/base_link.STL; visual mesh filename=~/Vibranium/baahubali/urdf/meshes/base_link.STL
- link linkOne: geometry collision mesh filename=~/Vibranium/baahubali/urdf/meshes/linkOne.STL; visual mesh filename=~/Vibranium/baahubali/urdf/meshes/linkOne.STL
- link linkTwo: geometry collision mesh filename=~/Vibranium/baahubali/urdf/meshes/linkTwo.STL; visual mesh filename=~/Vibranium/baahubali/urdf/meshes/linkTwo.STL
- link pitch: geometry collision mesh filename=~/Vibranium/baahubali/urdf/meshes/pitch.STL; visual mesh filename=~/Vibranium/baahubali/urdf/meshes/pitch.STL
- link roll: geometry collision mesh filename=~/Vibranium/baahubali/urdf/meshes/roll.STL; visual mesh filename=~/Vibranium/baahubali/urdf/meshes/roll.STL
- link turntable: geometry collision mesh filename=~/Vibranium/baahubali/urdf/ARMDIFF1/meshes/turntable.STL; visual mesh filename=~/Vibranium/baahubali/urdf/meshes/turntable.STL

Commit message: updated urdf

File: urdf/rerun_ARMDIFF.urdf (robot description, URDF)
Before this commit: robot ARMDIFF1, 6 links, 5 joints
Joints:
- joint linkOneJoint: origin xyz=0.08505 0 0.13572 rpy=0 2.17 0 -> xyz=0 0 0 rpy=0 0 0
- joint linkTwoJoint: origin xyz=-0.25101 0.0036996 0.34296 rpy=0 -1.84 0 -> xyz=0 0 0 rpy=0 0 0
