Commit message: 1. created new src folder

File: src/rerun_ARMDIFF.urdf (robot description, URDF)
Before this commit: robot ARMDIFF1, 6 links, 5 joints
Links:
- link base_link: geometry collision mesh filename=~/Vibranium/baahubali/src/meshes/base_link.STL; visual mesh filename=~/Vibranium/baahubali/src/meshes/base_link.STL
- link linkOne: geometry collision mesh filename=~/Vibranium/baahubali/src/meshes/linkOne.STL; visual mesh filename=~/Vibranium/baahubali/src/meshes/linkOne.STL
- link linkTwo: geometry collision mesh filename=~/Vibranium/baahubali/src/meshes/linkTwo.STL; visual mesh filename=~/Vibranium/baahubali/src/meshes/linkTwo.STL
- link pitch: geometry collision mesh filename=~/Vibranium/baahubali/src/meshes/pitch.STL; visual mesh filename=~/Vibranium/baahubali/src/meshes/pitch.STL
- link roll: geometry collision mesh filename=~/Vibranium/baahubali/src/meshes/roll.STL; visual mesh filename=~/Vibranium/baahubali/src/meshes/roll.STL
- link turntable: geometry collision mesh filename=~/Vibranium/baahubali/src/meshes/turntable.STL; visual mesh filename=~/Vibranium/baahubali/src/meshes/turntable.STL

File: urdf/.ipynb_checkpoints/ARMDIFF1-checkpoint.urdf (robot description, URDF)
Before this commit: robot ARMDIFF1, 6 links, 5 joints
Joints:
- joint linkOneJoint: origin xyz=0.08505 0 0.13572 rpy=0 2.17 0 -> xyz=0.08505 0 0.13572 rpy=0 0 0
- joint linkTwoJoint: origin xyz=-0.25101 0.0036996 0.34296 rpy=0 -1.84 0 -> xyz=-0.25101 0.0036996 0.34296 rpy=0 0 0
- joint rollJoint: origin xyz=0.017053 0 0.0065172 rpy=0.4 0 0 -> xyz=0.017053 0 0.0065172 rpy=0 0 0

Commit message: rerun changes

File: src/rerun_ARMDIFF.urdf (robot description, URDF)
Before this commit: robot ARMDIFF1, 6 links, 5 joints
Links:
- link base_link: geometry collision mesh filename=~/baahubali/src/meshes/base_link.STL; visual mesh filename=~/baahubali/src/meshes/base_link.STL
- link linkOne: geometry collision mesh filename=~/baahubali/src/meshes/linkOne.STL; visual mesh filename=~/baahubali/src/meshes/linkOne.STL
- link linkTwo: geometry collision mesh filename=~/baahubali/src/meshes/linkTwo.STL; visual mesh filename=~/baahubali/src/meshes/linkTwo.STL
- link pitch: geometry collision mesh filename=~/baahubali/src/meshes/pitch.STL; visual mesh filename=~/baahubali/src/meshes/pitch.STL
- link roll: geometry collision mesh filename=~/baahubali/src/meshes/roll.STL; visual mesh filename=~/baahubali/src/meshes/roll.STL
- link turntable: geometry collision mesh filename=~/baahubali/src/meshes/turntable.STL; visual mesh filename=~/baahubali/src/meshes/turntable.STL
